Commit message: poprawa błędów

File: lab2/urdf/static_robot.urdf (robot description, URDF)
Before this commit: robot robot, 3 links, 2 joints
Links:
- added link base_link; visual cylinder length=${base_l} radius=${base_r}
Joints:
- added joint base_to_link1: type fixed, parent base_link, child link_1, origin xyz=${props['i1']['j_xyz']} rpy=${props['i1']['j_rpy']}, axis 0 0 1

Commit message: odczyt parametrów z pliku yaml

File: lab2/urdf/static_robot.urdf (robot description, URDF)
Before this commit: robot robot, 4 links, 3 joints
Links:
- link base_link: geometry visual cylinder length=${param['base_l']} radius=${param['base_r']}
- link link_1: geometry visual box size=${props['i2']['l_len']} ${param['l_width']} ${param['l_heig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
- link link_2: geometry visual box size=${props['i3']['l_len']} ${param['l_width']} ${param['l_heig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
- link link_3: geometry visual cylinder length=${param['link3_len']} radius=${param['link3_rad']}
